File: ECG/ECG.kicad_sch (KiCad schematic)
At the start: 43 parts, among them J1 Conn_01x03, J2 Conn_01x03, J3 Conn_01x15, J4 Conn_01x15, J5 Conn_01x02, Q1 DMG2301L, Q2 T2N7002AK, Q3 T2N7002AK, Q4 T2N7002AK, Q5 T2N7002AK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

Commit message: tinkering with switching logic placements
Parts:
- added TP6: TestPoint, TestPoint:TestPoint_Keystone_5000-5004_Miniature, symbol Connector:TestPoint
Connections:
- net at U1.6 (SW): now also TP6.1
- net D3 renamed PWR_HOLD
Other:
- note added: "Battery connectors Screw terminal (5mm pitch) for 9V. Could solder a wired cap into the same footprint if preferred 2032 Holder for 3V always on"
- moved on the sheet: BT1, J5
Changed lines of the file:
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@@
 	(paper "A4")
 	(rectangle
+		(start 173.355 129.54)
+		(end 252.095 165.1)
+		(stroke
+			(width 0)
+			(type default)
+		)
+		(fill
+			(type none)
+		)
+	)
+	(rectangle
 		(start 123.19 129.54)
 		(end 173.355 195.58)
@@
 	(text "2032 Coin Cell\n"
 		(exclude_from_sim no)
-		(at 201.93 162.56 0)
+		(at 208.28 162.56 0)
 		(effects
 			(font
@@
 		)
 	)
+	(text "Battery connectors\n\nScrew terminal (5mm\npitch) for 9V.  Could\nsolder a wired cap \ninto the same \nfootprint if preferred\n\n2032 Holder for 3V \nalways on"
+		(exclude_from_sim no)
+		(at 186.182 147.066 0)
+		(effects
+			(font
+				(size 1.27 1.27)
+			)
+		)
+	)
 	(text "Should I add a shunt block or switch to turn on the processor in the event of a disaster?\n\n"
 		(exclude_from_sim no)
@@
 	(wire
 		(pts
-			(xy 223.52 146.05) (xy 220.345 146.05)
+			(xy 229.87 146.05) (xy 226.695 146.05)
 		)
 		(stroke
@@
 	(wire
 		(pts
-			(xy 220.345 146.05) (xy 220.345 154.305)
+			(xy 226.695 146.05) (xy 226.695 154.305)
 		)
 		(stroke
@@
 	(wire
 		(pts
-			(xy 220.345 139.065) (xy 220.345 143.51)
+			(xy 226.695 139.065) (xy 226.695 143.51)
 		)
 		(stroke
@@
 	(wire
 		(pts
-			(xy 223.52 143.51) (xy 220.345 143.51)
+			(xy 229.87 143.51) (xy 226.695 143.51)
 		)
 		(stroke
@@
 		)
 	)
-	(label "D3"
-		(at 248.285 77.47 0)
-		(effects
-			(font
-				(size 1.27 1.27)
-			)
-			(justify left bottom)
-		)
-	)
 	(label "A0"
 		(at 206.375 85.09 0)
@@
 		)
 	)
-	(label "D3"
+	(label "PWR_HOLD"
 		(at 160.655 160.655 0)
 		(effects
@@
 	(symbol
 		(lib_id "Connector_Generic:Conn_01x02")
-		(at 228.6 143.51 0)
+		(at 234.95 143.51 0)
 		(unit 1)
 		(exclude_from_sim no)
@@
 		(fields_autoplaced yes)
 		(property "Reference" "J5"
-			(at 231.14 143.5099 0)
+			(at 237.49 143.5099 0)
 			(effects
 				(font
@@
 		)
 		(property "Value" "Conn_01x02"
-			(at 231.14 146.0499 0)
+			(at 237.49 146.0499 0)
 			(effects
 				(font
@@
 		)
 		(property "Footprint" "ECG_Footprints:691137710002"
-			(at 228.6 143.51 0)
+			(at 234.95 143.51 0)
 			(effects
 				(font
@@
 		)
 		(property "Datasheet" "https://www.we-online.com/katalog/datasheet/691137710002.pdf"
-			(at 228.6 143.51 0)
+			(at 234.95 143.51 0)
 			(effects
 				(font
@@
 		)
 		(property "Description" "Generic connector, single row, 01x02, script generated (kicad-library-utils/schlib/autogen/connector/)"
-			(at 228.6 143.51 0)
+			(at 234.95 143.51 0)
 			(effects
 				(font
@@
 		)
 		(property "DigikeyPN" "732-10955-ND"
-			(at 228.6 143.51 0)
+			(at 234.95 143.51 0)
 			(effects
 				(font
@@
 	(symbol
 		(lib_id "EGC_Symbols:BS-3")
-		(at 201.295 146.685 270)
+		(at 207.645 146.685 270)
 		(unit 1)
 		(exclude_from_sim no)
@@
 		(fields_autoplaced yes)
 		(property "Reference" "BT1"
-			(at 205.74 145.4149 90)
+			(at 212.09 145.4149 90)
 			(effects
 				(font
@@
 		)
 		(property "Value" "BS-3"
-			(at 205.74 147.9549 90)
+			(at 212.09 147.9549 90)
 			(effects
 				(font
@@
 		)
 		(property "Footprint" "ECG_Footprints:BAT_BS-3"
-			(at 201.295 146.685 0)
+			(at 207.645 146.685 0)
 			(effects
 				(font
@@
 		)
 		(property "Datasheet" ""
-			(at 201.295 146.685 0)
+			(at 207.645 146.685 0)
 			(effects
 				(font
@@
 		)
 		(property "Description" ""
-			(at 201.295 146.685 0)
+			(at 207.645 146.685 0)
 			(effects
 				(font
@@
 		)
 		(property "PARTREV" "F"
-			(at 201.295 146.685 0)
+			(at 207.645 146.685 0)
 			(effects
 				(font
@@
 		)
 		(property "STANDARD" "Manufacturer recommendations"
-			(at 201.295 146.685 0)
+			(at 207.645 146.685 0)
 			(effects
 				(font
@@
 		)
 		(property "MAXIMUM_PACKAGE_HEIGHT" "6.75mm"
-			(at 201.295 146.685 0)
+			(at 207.645 146.685 0)
 			(effects
 				(font
@@
 		)
 		(property "MANUFACTURER" "MPD"
-			(at 201.295 146.685 0)
+			(at 207.645 146.685 0)
 			(effects
 				(font
@@
 	(symbol
 		(lib_id "power:+3V0")
-		(at 201.295 139.065 0)
+		(at 207.645 139.065 0)
 		(unit 1)
 		(exclude_from_sim no)
@@
 		(fields_autoplaced yes)
 		(property "Reference" "#PWR034"
-			(at 201.295 142.875 0)
+			(at 207.645 142.875 0)
 			(effects
 				(font
@@
 		)
 		(property "Value" "+3V0"
-			(at 201.295 133.985 0)
+			(at 207.645 133.985 0)
 			(effects
 				(font
@@
 		)
 		(property "Footprint" ""
-			(at 201.295 139.065 0)
+			(at 207.645 139.065 0)
 			(effects
 				(font
@@
 		)
 		(property "Datasheet" ""
-			(at 201.295 139.065 0)
+			(at 207.645 139.065 0)
 			(effects
 				(font
@@
 		)
 		(property "Description" "Power symbol creates a global label with name \"+3V0\""
-			(at 201.295 139.065 0)
+			(at 207.645 139.065 0)
 			(effects
 				(font
@@
 	(symbol
 		(lib_id "power:+9V")
-		(at 220.345 139.065 0)
+		(at 226.695 139.065 0)
 		(unit 1)
 		(exclude_from_sim no)
@@
 		(dnp no)
 		(property "Reference" "#PWR035"
-			(at 220.345 142.875 0)
+			(at 226.695 142.875 0)
 			(effects
 				(font
@@
 		)
 		(property "Value" "+9V"
-			(at 220.345 134.62 90)
+			(at 226.695 134.62 90)
 			(effects
 				(font
@@
 		)
 		(property "Footprint" ""
-			(at 220.345 139.065 0)
+			(at 226.695 139.065 0)
 			(effects
 				(font
@@
 		)
 		(property "Datasheet" ""
-			(at 220.345 139.065 0)
+			(at 226.695 139.065 0)
 			(effects
 				(font
@@
 		)
 		(property "Description" "Power symbol creates a global label with name \"+9V\""
-			(at 220.345 139.065 0)
+			(at 226.695 139.065 0)
 			(effects
 				(font
@@
 	)
 	(symbol
+		(lib_id "Connector:TestPoint")
+		(at 103.505 90.17 180)
+		(unit 1)
+		(exclude_from_sim no)
+		(in_bom yes)
+		(on_board yes)
+		(dnp no)
+		(fields_autoplaced yes)
+		(property "Reference" "TP6"
+			(at 106.045 93.4719 0)
+			(effects
+				(font
+					(size 1.27 1.27)
+				)
+				(justify right)
+			)
+		)
+		(property "Value" "TestPoint"
+			(at 102.2351 95.885 90)
+			(effects
+				(font
+					(size 1.27 1.27)
+				)
+				(justify left)
+				(hide yes)
+			)
+		)
+		(property "Footprint" "TestPoint:TestPoint_Keystone_5000-5004_Miniature"
+			(at 98.425 90.17 0)
+			(effects
+				(font
+					(size 1.27 1.27)
+				)
+				(hide yes)
+			)
+		)
+		(property "Datasheet" "~"
+			(at 98.425 90.17 0)
+			(effects
+				(font
+					(size 1.27 1.27)
+				)
+				(hide yes)
+			)
+		)
+		(property "Description" "test point"
+			(at 103.505 90.17 0)
+			(effects
+				(font
+					(size 1.27 1.27)
+				)
+				(hide yes)
+			)
+		)
+		(pin "1"
+		)
+		(instances
+			(project "ECG"
+				(path "/e3a79443-8349-4546-8b4f-331bcc551083"
+					(reference "TP6")
+					(unit 1)
+				)
+			)
+		)
+	)
+	(symbol
 		(lib_id "power:GND")
 		(at 62.23 180.34 0)
@@
 	(symbol
 		(lib_id "power:GND")
-		(at 201.295 154.305 0)
+		(at 207.645 154.305 0)
 		(unit 1)
 		(exclude_from_sim no)
@@
 		(fields_autoplaced yes)
 		(property "Reference" "#PWR07"
-			(at 201.295 160.655 0)
+			(at 207.645 160.655 0)
 			(effects
 				(font
@@
 		)
 		(property "Value" "GND"
-			(at 201.295 159.385 0)
+			(at 207.645 159.385 0)
 			(effects
 				(font
@@
 		)
 		(property "Footprint" ""
-			(at 201.295 154.305 0)
+			(at 207.645 154.305 0)
 			(effects
 				(font
@@
 		)
 		(property "Datasheet" ""
-			(at 201.295 154.305 0)
+			(at 207.645 154.305 0)
 			(effects
 				(font
@@
 		)
 		(property "Description" "Power symbol creates a global label with name \"GND\" , ground"
-			(at 201.295 154.305 0)
+			(at 207.645 154.305 0)
 			(effects
 				(font
@@
 	(symbol
 		(lib_id "power:GND")
-		(at 220.345 154.305 0)
+		(at 226.695 154.305 0)
 		(unit 1)
 		(exclude_from_sim no)
@@
 		(fields_autoplaced yes)
 		(property "Reference" "#PWR010"
-			(at 220.345 160.655 0)
+			(at 226.695 160.655 0)
 			(effects
 				(font
@@
 		)
 		(property "Value" "GND"
-			(at 220.345 159.385 0)
+			(at 226.695 159.385 0)
 			(effects
 				(font
@@
 		)
 		(property "Footprint" ""
-			(at 220.345 154.305 0)
+			(at 226.695 154.305 0)
 			(effects
 				(font
@@
 		)
 		(property "Datasheet" ""
-			(at 220.345 154.305 0)
+			(at 226.695 154.305 0)
 			(effects
 				(font
@@
 		)
 		(property "Description" "Power symbol creates a global label with name \"GND\" , ground"
-			(at 220.345 154.305 0)
+			(at 226.695 154.305 0)
 			(effects
 				(font

Commit message: WIP
first edits
Parts:
- added D1: LED, LED_SMD:LED_0603_1608Metric, symbol Device:LED
- added JP1: SolderJumper_2_Open, Jumper:SolderJumper-2_P1.3mm_Open_RoundedPad1.0x1.5mm, symbol Jumper:SolderJumper_2_Open
- added R1: 1k, Resistor_SMD:R_0603_1608Metric, symbol Device:R_Small_US
Connections:
- net GND: now also JP1.1 (A)
- net RLD: now also C5.2, R10.2, U1.5 (RLD); no longer J2.1 (Pin_1), R10.1, TP5.1
- net at R13.2, R14.1, U1.10 (OUT): now also D1.2 (A)
- new net: JP1.2 (B), R1.2
- new net: D1.1 (K), R1.1
- new net RL: J2.1 (Pin_1), R10.1, TP5.1

Commit message: WIP2
new positions
Parts:
- C5: footprint Capacitor_THT:C_Rect_L7.2mm_W5.5mm_P5.00mm_FKS2_FKP2_MKS2_MKP2 -> Capacitor_SMD:C_0603_1608Metric
- R12, R13: footprint Resistor_THT:R_Axial_DIN0207_L6.3mm_D2.5mm_P2.54mm_Vertical -> Resistor_SMD:R_0603_1608Metric
Changed lines of the file:
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@@
 			)
 		)
-		(property "Footprint" "Resistor_THT:R_Axial_DIN0207_L6.3mm_D2.5mm_P2.54mm_Vertical"
+		(property "Footprint" "Resistor_SMD:R_0603_1608Metric"
 			(at 121.285 95.25 0)
 			(effects
@@
 			)
 		)
-		(property "Footprint" "Capacitor_THT:C_Rect_L7.2mm_W5.5mm_P5.00mm_FKS2_FKP2_MKS2_MKP2"
+		(property "Footprint" "Capacitor_SMD:C_0603_1608Metric"
 			(at 95.885 80.01 0)
 			(effects
@@
 			)
 		)
-		(property "Footprint" "Resistor_THT:R_Axial_DIN0207_L6.3mm_D2.5mm_P2.54mm_Vertical"
+		(property "Footprint" "Resistor_SMD:R_0603_1608Metric"
 			(at 116.205 95.25 0)
 			(effects

Commit message: WIPmorning1
switch added
Parts:
- added C21: DNP, Capacitor_THT:C_Rect_L7.2mm_W5.5mm_P5.00mm_FKS2_FKP2_MKS2_MKP2, symbol Device:C_Small
- added R22: DNP, Resistor_THT:R_Axial_DIN0207_L6.3mm_D2.5mm_P2.54mm_Vertical, symbol Device:R_Small_US
- added SW1: SW_Slide_DPDT, symbol Switch:SW_Slide_DPDT
Connections:
- net +3V0: now also SW1.1 (A); no longer BT1.+
- net +9V: now also SW1.6 (C); no longer J5.1 (Pin_1)
- net P1: now also R22.1
- net at C6.1, R11.2, U1.7 (OPAMP+): now also C21.1, R22.2
- net at C6.2, R12.1, U1.8 (REFOUT): now also C21.2
- new net: J5.1 (Pin_1), SW1.5 (B)
- new net: BT1.+, SW1.2 (B)
Other:
- moved on the sheet: BT1, J5

Commit message: WIPmorn2
SBD
Parts:
- added D3: D_Schottky_Small_Filled, Diode_SMD:D_SOD-123F, symbol Device:D_Schottky_Small_Filled
Connections:
- net at J5.1 (Pin_1): now also D3.2 (A); no longer SW1.5 (B)
- new net: D3.1 (K), SW1.5 (B)
Other:
- moved on the sheet: SW1
Changed lines of the file:
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@@
 	(wire
 		(pts
-			(xy 226.06 142.24) (xy 226.06 137.16)
+			(xy 226.06 138.43) (xy 226.06 137.16)
 		)
 		(stroke
@@
 	(wire
 		(pts
-			(xy 226.06 147.32) (xy 223.52 147.32)
+			(xy 224.155 143.51) (xy 227.33 143.51)
 		)
 		(stroke
@@
 	(wire
 		(pts
-			(xy 213.36 142.24) (xy 210.82 142.24)
+			(xy 213.995 138.43) (xy 210.82 138.43)
 		)
 		(stroke
@@
 	(wire
 		(pts
-			(xy 226.06 143.51) (xy 232.41 143.51)
-		)
-		(stroke
-			(width 0)
-			(type default)
-		)
-	)
-	(wire
-		(pts
 			(xy 39.37 56.515) (xy 39.37 82.55)
 		)
@@
 	(wire
 		(pts
-			(xy 210.82 142.24) (xy 210.82 137.16)
+			(xy 210.82 138.43) (xy 210.82 137.16)
 		)
 		(stroke
@@
 	(wire
 		(pts
-			(xy 226.06 143.51) (xy 226.06 147.32)
-		)
-		(stroke
-			(width 0)
-			(type default)
-		)
-	)
-	(wire
-		(pts
 			(xy 250.19 113.03) (xy 250.19 120.65)
 		)
@@
 	(wire
 		(pts
-			(xy 209.55 147.32) (xy 213.36 147.32)
+			(xy 209.55 143.51) (xy 213.995 143.51)
 		)
 		(stroke
@@
 	(wire
 		(pts
-			(xy 223.52 142.24) (xy 226.06 142.24)
+			(xy 224.155 138.43) (xy 226.06 138.43)
 		)
 		(stroke
@@
 	(wire
 		(pts
-			(xy 209.55 138.43) (xy 209.55 147.32)
+			(xy 209.55 138.43) (xy 209.55 143.51)
 		)
 		(stroke
@@
 	)
 	(symbol
+		(lib_id "Device:D_Schottky_Small_Filled")
+		(at 229.87 143.51 0)
+		(unit 1)
+		(exclude_from_sim no)
+		(in_bom yes)
+		(on_board yes)
+		(dnp no)
+		(fields_autoplaced yes)
+		(property "Reference" "D3"
+			(at 229.616 137.795 0)
+			(effects
+				(font
+					(size 1.27 1.27)
+				)
+			)
+		)
+		(property "Value" "D_Schottky_Small_Filled"
+			(at 229.616 140.335 0)
+			(effects
+				(font
+					(size 1.27 1.27)
+				)
+			)
+		)
+		(property "Footprint" "Diode_SMD:D_SOD-123F"
+			(at 229.87 143.51 90)
+			(effects
+				(font
+					(size 1.27 1.27)
+				)
+				(hide yes)
+			)
+		)
+		(property "Datasheet" "~"
+			(at 229.87 143.51 90)
+			(effects
+				(font
+					(size 1.27 1.27)
+				)
+				(hide yes)
+			)
+		)
+		(property "Description" "Schottky diode, small symbol, filled shape"
+			(at 229.87 143.51 0)
+			(effects
+				(font
+					(size 1.27 1.27)
+				)
+				(hide yes)
+			)
+		)
+		(pin "1"
+		)
+		(pin "2"
+		)
+		(instances
+			(project ""
+				(path "/e3a79443-8349-4546-8b4f-331bcc551083"
+					(reference "D3")
+					(unit 1)
+				)
+			)
+		)
+	)
+	(symbol
 		(lib_id "Transistor_FET:T2N7002AK")
 		(at 74.93 167.005 0)
@@
 	(symbol
 		(lib_id "Switch:SW_Slide_DPDT")
-		(at 218.44 147.32 0)
+		(at 219.075 143.51 0)
 		(unit 1)
 		(exclude_from_sim no)
@@
 		(fields_autoplaced yes)
 		(property "Reference" "SW1"
-			(at 218.44 137.16 0)
+			(at 219.075 133.35 0)
 			(effects
 				(font
@@
 		)
 		(property "Value" "SW_Slide_DPDT"
-			(at 218.44 139.7 0)
+			(at 219.075 135.89 0)
 			(effects
 				(font
@@
 		)
 		(property "Footprint" ""
-			(at 232.41 142.24 0)
+			(at 233.045 138.43 0)
 			(effects
 				(font
@@
 		)
 		(property "Datasheet" "~"
-			(at 218.44 147.32 0)
+			(at 219.075 143.51 0)
 			(effects
 				(font
@@
 		)
 		(property "Description" "Slide Switch, dual pole double throw"
-			(at 218.44 147.32 0)
+			(at 219.075 143.51 0)
 			(effects
 				(font

Commit message: R22
want layout update
Other:
- moved on the sheet: C21
Changed lines of the file:
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@@
 	)
 	(junction
-		(at 106.68 95.25)
-		(diameter 0)
-		(color 0 0 0 0)
-	)
-	(junction
 		(at 41.91 167.005)
 		(diameter 0)
@@
 	)
 	(junction
-		(at 113.665 95.25)
+		(at 72.39 153.035)
 		(diameter 0)
 		(color 0 0 0 0)
 	)
 	(junction
-		(at 72.39 153.035)
+		(at 39.37 82.55)
 		(diameter 0)
 		(color 0 0 0 0)
 	)
 	(junction
-		(at 39.37 82.55)
+		(at 55.245 67.31)
 		(diameter 0)
 		(color 0 0 0 0)
 	)
 	(junction
-		(at 55.245 67.31)
+		(at 113.665 95.25)
 		(diameter 0)
 		(color 0 0 0 0)
@@
 	(wire
 		(pts
-			(xy 113.665 95.25) (xy 114.3 95.25)
-		)
-		(stroke
-			(width 0)
-			(type default)
-		)
-	)
-	(wire
-		(pts
 			(xy 247.015 97.79) (xy 252.095 97.79)
 		)
@@
 	(wire
 		(pts
-			(xy 113.03 104.14) (xy 113.03 95.25)
-		)
-		(stroke
-			(width 0)
-			(type default)
-		)
-	)
-	(wire
-		(pts
 			(xy 204.47 97.79) (xy 211.455 97.79)
 		)
@@
 	(wire
 		(pts
+			(xy 113.665 90.17) (xy 113.665 95.25)
+		)
+		(stroke
+			(width 0)
+			(type default)
+		)
+	)
+	(wire
+		(pts
 			(xy 39.37 56.515) (xy 39.37 82.55)
 		)
@@
 	(wire
 		(pts
+			(xy 108.585 95.25) (xy 108.585 102.235)
+		)
+		(stroke
+			(width 0)
+			(type default)
+		)
+	)
+	(wire
+		(pts
 			(xy 204.47 100.33) (xy 211.455 100.33)
 		)
@@
 	(wire
 		(pts
-			(xy 113.03 95.25) (xy 113.665 95.25)
-		)
-		(stroke
-			(width 0)
-			(type default)
-		)
-	)
-	(wire
-		(pts
 			(xy 199.39 138.43) (xy 209.55 138.43)
 		)
@@
 	(wire
 		(pts
-			(xy 107.95 104.14) (xy 106.68 104.14)
-		)
-		(stroke
-			(width 0)
-			(type default)
-		)
-	)
-	(wire
-		(pts
 			(xy 204.47 90.17) (xy 211.455 90.17)
 		)
@@
 	(wire
 		(pts
-			(xy 92.71 95.25) (xy 106.68 95.25)
+			(xy 113.665 95.25) (xy 113.665 102.235)
 		)
 		(stroke
@@
 	(wire
 		(pts
-			(xy 113.665 95.25) (xy 113.665 90.17)
-		)
-		(stroke
-			(width 0)
-			(type default)
-		)
-	)
-	(wire
-		(pts
 			(xy 85.725 85.725) (xy 85.725 86.995)
 		)
@@
 	(wire
 		(pts
-			(xy 108.585 95.25) (xy 106.68 95.25)
+			(xy 92.71 95.25) (xy 108.585 95.25)
 		)
 		(stroke
@@
 	(wire
 		(pts
-			(xy 106.68 104.14) (xy 106.68 95.25)
-		)
-		(stroke
-			(width 0)
-			(type default)
-		)
-	)
-	(wire
-		(pts
 			(xy 43.815 67.31) (xy 36.83 67.31)
 		)
@@
 	(symbol
 		(lib_id "Device:C_Small")
-		(at 110.49 104.14 90)
+		(at 111.125 102.235 90)
 		(unit 1)
 		(exclude_from_sim no)
@@
 		(dnp no)
 		(property "Reference" "C21"
-			(at 110.236 106.934 90)
+			(at 110.871 105.029 90)
 			(effects
 				(font
@@
 		)
 		(property "Value" "DNP"
-			(at 110.49 108.712 90)
+			(at 111.125 106.807 90)
 			(effects
 				(font
@@
 		)
 		(property "Footprint" "Capacitor_THT:C_Rect_L7.2mm_W5.5mm_P5.00mm_FKS2_FKP2_MKS2_MKP2"
-			(at 110.49 104.14 0)
+			(at 111.125 102.235 0)
 			(effects
 				(font
@@
 		)
 		(property "Datasheet" "~"
-			(at 110.49 104.14 0)
+			(at 111.125 102.235 0)
 			(effects
 				(font
@@
 		)
 		(property "Description" "Unpolarized capacitor, small symbol"
-			(at 110.49 104.14 0)
+			(at 111.125 102.235 0)
 			(effects
 				(font

Commit message: Done for Friday
See you Monday. Parts connected and snugged up.
Parts:
- added C22: DNP, Capacitor_THT:C_Rect_L7.2mm_W5.5mm_P5.00mm_FKS2_FKP2_MKS2_MKP2, symbol Device:C_Small
Connections:
- net P1: now also C22.1
- net at C2.2, R5.2, U1.20 (HPSENSE): now also C22.2
Changed lines of the file:
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@@
 	)
 	(junction
+		(at 93.345 62.23)
+		(diameter 0)
+		(color 0 0 0 0)
+	)
+	(junction
 		(at 118.745 95.25)
 		(diameter 0)
@@
 	)
 	(junction
+		(at 93.345 50.8)
+		(diameter 0)
+		(color 0 0 0 0)
+	)
+	(junction
 		(at 129.54 95.25)
 		(diameter 0)
@@
 	(wire
 		(pts
+			(xy 93.345 50.8) (xy 103.505 50.8)
+		)
+		(stroke
+			(width 0)
+			(type default)
+		)
+	)
+	(wire
+		(pts
 			(xy 128.27 158.115) (xy 140.97 158.115)
 		)
@@
 	(wire
 		(pts
-			(xy 85.725 50.8) (xy 103.505 50.8)
+			(xy 85.725 50.8) (xy 93.345 50.8)
 		)
 		(stroke
@@
 	(wire
 		(pts
+			(xy 93.345 50.8) (xy 93.345 53.34)
+		)
+		(stroke
+			(width 0)
+			(type default)
+		)
+	)
+	(wire
+		(pts
 			(xy 48.895 72.39) (xy 52.07 72.39)
 		)
@@
 	(wire
 		(pts
-			(xy 85.725 62.23) (xy 95.885 62.23)
+			(xy 85.725 62.23) (xy 93.345 62.23)
 		)
 		(stroke
@@
 	(wire
 		(pts
+			(xy 93.345 62.23) (xy 95.885 62.23)
+		)
+		(stroke
+			(width 0)
+			(type default)
+		)
+	)
+	(wire
+		(pts
 			(xy 72.39 153.035) (xy 76.835 153.035)
 		)
@@
 	(wire
 		(pts
+			(xy 93.345 58.42) (xy 93.345 62.23)
+		)
+		(stroke
+			(width 0)
+			(type default)
+		)
+	)
+	(wire
+		(pts
 			(xy 168.275 142.875) (xy 158.115 142.875)
 		)
@@
 					(unit 1)
 				)
+			)
+		)
+	)
+	(symbol
+		(lib_id "Device:C_Small")
+		(at 93.345 55.88 0)
+		(mirror x)
+		(unit 1)
+		(exclude_from_sim no)
+		(in_bom yes)
+		(on_board yes)
+		(dnp no)
+		(property "Reference" "C22"
+			(at 90.805 54.6035 0)
+			(effects
+				(font
+					(size 1.27 1.27)
+				)
+				(justify right)
+			)
+		)
+		(property "Value" "DNP"
+			(at 90.805 57.1435 0)
+			(effects
+				(font
+					(size 1.27 1.27)
+				)
+				(justify right)
+			)
+		)
+		(property "Footprint" "Capacitor_THT:C_Rect_L7.2mm_W5.5mm_P5.00mm_FKS2_FKP2_MKS2_MKP2"
+			(at 93.345 55.88 0)
+			(effects
+				(font
+					(size 1.27 1.27)
+				)
+				(hide yes)
+			)
+		)
+		(property "Datasheet" "~"
+			(at 93.345 55.88 0)
+			(effects
+				(font
+					(size 1.27 1.27)
+				)
+				(hide yes)
+			)
+		)
+		(property "Description" "Unpolarized capacitor, small symbol"
+			(at 93.345 55.88 0)
+			(effects
+				(font
+					(size 1.27 1.27)
+				)
+				(hide yes)
+			)
+		)
+		(pin "1"
+		)
+		(pin "2"
+		)
+		(instances
+			(project "ECG"
+				(path "/e3a79443-8349-4546-8b4f-331bcc551083"
+					(reference "C22")
+					(unit 1)
+				)
