File: ECG/ECG.kicad_sch (KiCad schematic)
At the start: 86 parts, among them J1 Conn_01x03, J10 Socket 1x15, J11 Shunt block, J12 Shunt block, J13 Shunt block, J14 Shunt block, J15 Shunt block, J2 Conn_01x03, J3 Conn_01x15, J4 Conn_01x15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

Commit message: wip
Parts:
- J10: footprint Connector_PinHeader_2.54mm:PinHeader_1x15_P2.54mm_Vertical -> Connector_PinSocket_2.54mm:PinSocket_1x15_P2.54mm_Vertical; now fitted
- J11, J12, J13, J14, J15, J9, TP1, TP2, TP3, TP4, TP5, TP6, TP7, TP8: now fitted
- J8: footprint Connector_PinSocket_2.54mm:PinSocket_2x05_P2.54mm_Vertical -> Connector_PinHeader_2.54mm:PinHeader_2x05_P2.54mm_Vertical
Connections:
- net GND: now also J5.1 (Pin_1); no longer J5.2 (Pin_2)
- net at D3.2 (A): now also J5.2 (Pin_2); no longer J5.1 (Pin_1)
Changed lines of the file:
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@@
 			)
 		)
-		(property "Footprint" "Connector_PinSocket_2.54mm:PinSocket_2x05_P2.54mm_Vertical"
+		(property "Footprint" "Connector_PinHeader_2.54mm:PinHeader_2x05_P2.54mm_Vertical"
 			(at 53.34 168.91 0)
 			(effects
@@
 	(symbol
 		(lib_id "Connector_Generic:Conn_01x02")
-		(at 252.73 143.51 0)
+		(at 252.73 146.05 0)
+		(mirror x)
 		(unit 1)
 		(exclude_from_sim no)
@@
 		(on_board yes)
 		(dnp no)
-		(fields_autoplaced yes)
 		(property "Reference" "J5"
-			(at 255.905 144.7799 0)
+			(at 256.032 145.796 0)
 			(effects
 				(font
 					(size 1.27 1.27)
 				)
-				(justify left)
 			)
 		)
 		(property "Value" "Conn_01x02"
-			(at 255.27 146.0499 0)
+			(at 255.27 143.5101 0)
 			(effects
 				(font
@@
 		)
 		(property "Footprint" "ECG_Footprints:691137710002"
-			(at 252.73 143.51 0)
+			(at 252.73 146.05 0)
 			(effects
 				(font
@@
 		)
 		(property "Datasheet" "https://www.we-online.com/katalog/datasheet/691137710002.pdf"
-			(at 252.73 143.51 0)
+			(at 252.73 146.05 0)
 			(effects
 				(font
@@
 		)
 		(property "Description" "Generic connector, single row, 01x02, script generated (kicad-library-utils/schlib/autogen/connector/)"
-			(at 252.73 143.51 0)
+			(at 252.73 146.05 0)
 			(effects
 				(font
@@
 		)
 		(property "DigikeyPN" "36-232-ND"
-			(at 252.73 143.51 0)
+			(at 252.73 146.05 0)
 			(effects
 				(font
@@
 		)
 		(property "Sim.Device" ""
-			(at 252.73 143.51 0)
+			(at 252.73 146.05 0)
 			(effects
 				(font
@@
 		)
 		(property "Sim.Pins" ""
-			(at 252.73 143.51 0)
+			(at 252.73 146.05 0)
 			(effects
 				(font
@@
 		)
 		(property "AlternatePart" "732-10955-ND (TerminalBlock)"
-			(at 252.73 143.51 0)
+			(at 252.73 146.05 0)
 			(effects
 				(font
@@
 		)
 		(property "LCSC" ""
-			(at 252.73 143.51 0)
+			(at 252.73 146.05 0)
 			(effects
 				(font
@@
 		)
 		(property "Manufacturer_PN" ""
-			(at 252.73 143.51 0)
+			(at 252.73 146.05 0)
 			(effects
 				(font
@@
 		(in_bom yes)
 		(on_board yes)
-		(dnp yes)
+		(dnp no)
 		(property "Reference" "TP8"
 			(at 143.51 103.505 90)
@@
 		(in_bom yes)
 		(on_board yes)
-		(dnp yes)
+		(dnp no)
 		(property "Reference" "TP5"
 			(at 37.338 51.562 0)
@@
 				)
 				(justify left)
+				(hide yes)
 			)
 		)
@@
 		(in_bom yes)
 		(on_board no)
-		(dnp yes)
+		(dnp no)
 		(fields_autoplaced yes)
 		(property "Reference" "J13"
@@
 		(in_bom yes)
 		(on_board no)
-		(dnp yes)
+		(dnp no)
 		(fields_autoplaced yes)
 		(property "Reference" "J15"
@@
 		(in_bom yes)
 		(on_board yes)
-		(dnp yes)
+		(dnp no)
 		(property "Reference" "TP7"
 			(at 114.3 108.585 90)
@@
 		(in_bom yes)
 		(on_board yes)
-		(dnp yes)
+		(dnp no)
 		(property "Reference" "TP2"
 			(at 149.86 76.835 90)
@@
 		(in_bom yes)
 		(on_board yes)
-		(dnp yes)
+		(dnp no)
 		(property "Reference" "TP1"
 			(at 150.495 81.915 90)
@@
 		(in_bom yes)
 		(on_board yes)
-		(dnp yes)
+		(dnp no)
 		(property "Reference" "TP3"
 			(at 50.292 51.562 0)
@@
 		(in_bom yes)
 		(on_board no)
-		(dnp yes)
+		(dnp no)
 		(fields_autoplaced yes)
 		(property "Reference" "J14"
@@
 		(in_bom yes)
 		(on_board yes)
-		(dnp yes)
+		(dnp no)
 		(property "Reference" "TP4"
 			(at 53.848 51.562 0)
@@
 		(in_bom yes)
 		(on_board no)
-		(dnp yes)
+		(dnp no)
 		(fields_autoplaced yes)
 		(property "Reference" "J10"
@@
 			)
 		)
-		(property "Footprint" "Connector_PinHeader_2.54mm:PinHeader_1x15_P2.54mm_Vertical"
+		(property "Footprint" "Connector_PinSocket_2.54mm:PinSocket_1x15_P2.54mm_Vertical"
 			(at 184.15 37.465 0)
 			(effects
@@
 		(in_bom yes)
 		(on_board no)
-		(dnp yes)
+		(dnp no)
 		(fields_autoplaced yes)
 		(property "Reference" "J11"
@@
 		(in_bom yes)
 		(on_board yes)
-		(dnp yes)
+		(dnp no)
 		(fields_autoplaced yes)
 		(property "Reference" "TP6"
@@
 		(in_bom yes)
 		(on_board no)
-		(dnp yes)
+		(dnp no)
 		(fields_autoplaced yes)
 		(property "Reference" "J9"
@@
 		(in_bom yes)
 		(on_board no)
-		(dnp yes)
+		(dnp no)
 		(fields_autoplaced yes)
 		(property "Reference" "J12"
